File: 2x5-1-27-to-2x5-2-54/2x5-1-27-to-2x5-2-54.kicad_pcb (KiCad board)
At the start: 2 copper layers, 30 x 15 mm, 4 parts, among them J1 Conn_02x05_Odd_Even, J2 Conn_02x05_Odd_Even

Commit message: single gerber
Other:
- board text removed: "ADAP-1.27-2-54"
Changed lines of the file:
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@@
     (effects (font (size 1 1) (thickness 0.15)))
   )
-  (gr_text "ADAP-1.27-2-54" (at 108.22 113.665) (layer "F.SilkS")
+  (gr_text "ADAP-1.27-2.54" (at 108.22 113.665) (layer "F.SilkS")
     (effects (font (size 1 1) (thickness 0.15)))
   )
